Commit message: Update tof_vlp16_rover.urdf

File: cartographer_ros/urdf/tof_vlp16_rover.urdf (robot description, URDF)
Before this commit: robot xsens_cartographer_backpack_3d, 6 links, 5 joints
Joints:
- joint l_tof_camera_link_joint: origin xyz=.232 -.102 .064 rpy=0 -1.18 -1.57 -> xyz=.232 .102 .064 rpy=0 -1.169 -1.57
- joint r_tof_camera_link_joint: origin xyz=.33 .102 .064 rpy=0 -1.18 1.57 -> xyz=.33 -.102 .064 rpy=0 -1.169 1.57
