Commit message: first commit

File: cartographer_ros/urdf/backpack_2d_ori.urdf (robot description, URDF)
Before this commit: robot cartographer_backpack_2d, 2 links, 1 joints
Joints:
- removed joint laser_link_joint
- added joint laser_baselink: type fixed, parent base_link, child laser, origin xyz=0. 0 0.0
