Commit message: Add code to allow offline processing of 2D Cartographer bags.
Fixes waiting for transforms to be published, adds support for multi-echo
laser scans, sets default values for the submap topic and query for the
RViz plugin.

File: cartographer_ros/urdf/backpack_2d.urdf (robot description, URDF)
Before this commit: robot cartographer_ros, 4 links, 3 joints
Links:
- removed link /base_footprint
- removed link /horizontal_laser_link
- removed link /imu_link
- removed link /vertical_laser_link
- added link base_link; visual box size=0.03 0.4 0.8
- added link horizontal_laser_link; visual cylinder length=0.09 radius=0.03
- added link imu_link; visual box size=0.055 0.055 0.02
- added link vertical_laser_link; visual cylinder length=0.09 radius=0.03
Joints:
- joint base_link_joint: child /imu_link -> imu_link; parent /base_footprint -> base_link
- joint horizontal_laser_link_joint: child /horizontal_laser_link -> horizontal_laser_link; parent /imu_link -> base_link
- joint vertical_laser_link_joint: child /vertical_laser_link -> vertical_laser_link; parent /imu_link -> base_link

Commit message: Addresses code review comments.

File: cartographer_ros/urdf/backpack_2d.urdf (robot description, URDF)
Before this commit: robot cartographer_ros, 4 links, 3 joints
Joints:
- removed joint base_link_joint
- added joint imu_link_joint: type fixed, parent base_link, child imu_link, origin xyz=0 0 0 rpy=0 0 3.1416

Commit message: LiDAR turn

File: cartographer_ros/urdf/backpack_2d.urdf (robot description, URDF)
Before this commit: robot cartographer_backpack_2d, 2 links, 1 joints
Joints:
- joint laser_link_joint: origin xyz=0. 0 0.0 -> xyz=0. 0 0.0 rpy=0 0 3.14159
